Commit message: tuned pid controller, gets to the desired position within 1 sec

File: urdf/stand_chest.xacro (robot description, xacro)
@@ -15,5 +15,5 @@
   <child link="chest_1"/>
   <axis xyz="0.0 0.0 1.0"/>
-  <limit upper="0.47" lower="0.00" effort="1000000" velocity="100000"/>
+  <limit upper="0.47" lower="0.00" effort="1000000" velocity="0.5"/>
 </joint>
 <link name="stand">

Commit message: added the freight to the model to connect these two together. Will ned to try and connect the robot to the actual base from the fright package

File: urdf/stand_chest.xacro (robot description, xacro)
@@ -4,10 +4,18 @@
 <xacro:include filename="$(find stand_chest_description)/urdf/stand_chest.trans" />
 <xacro:include filename="$(find stand_chest_description)/urdf/stand_chest.gazebo" />
-<link name="base_link"></link>
+<xacro:include filename="$(find stand_chest_description)/urdf/freight.gazebo" />
+<xacro:include filename="$(find stand_chest_description)/urdf/freight.xacro" />
+<!-- <link name="base_link"></link> -->
 <joint name="base_link_to_stand" type="fixed">
-  <origin xyz="0.0 0.0 0.0" rpy="0 0 0"/>
+  <origin xyz="-0.1 0.0 0.357425" rpy="0 0 0"/>
   <parent link="base_link"/>
   <child link="stand"/>
 </joint>
+<!-- <joint name="torso_fixed_joint" type="fixed">
+    <origin rpy="-6.12303176911189E-17 0 0" xyz="-0.086875 0 0.377425" />
+    <parent link="base_link" />
+    <child link="torso_fixed_link" />
+    <axis xyz="0 1 0" />
+</joint> -->
 <joint name="Zaxis" type="prismatic">
   <origin xyz="-0.082038 0.000502 0.303534" rpy="0 0 0"/>

Commit message: modified the gazebo launch to load with or without the mobile base

File: urdf/stand_chest.xacro (robot description, xacro)
@@ -4,17 +4,4 @@
 <xacro:include filename="$(find stand_chest_description)/urdf/stand_chest.trans" />
 <xacro:include filename="$(find stand_chest_description)/urdf/stand_chest.gazebo" />
-<xacro:include filename="$(find fetch_gazebo)/robots/freight.gazebo.xacro" />
-<!-- <link name="base_link"></link> -->
-<joint name="base_link_to_stand" type="fixed">
-  <origin xyz="-0.1 0.0 0.357425" rpy="0 0 0"/>
-  <parent link="base_link"/>
-  <child link="stand"/>
-</joint>
-<!-- <joint name="torso_fixed_joint" type="fixed">
-    <origin rpy="-6.12303176911189E-17 0 0" xyz="-0.086875 0 0.377425" />
-    <parent link="base_link" />
-    <child link="torso_fixed_link" />
-    <axis xyz="0 1 0" />
-</joint> -->
 <joint name="Zaxis" type="prismatic">
   <origin xyz="-0.082038 0.000502 0.303534" rpy="0 0 0"/>

Commit message: -

File: urdf/stand_chest.xacro (robot description, xacro)
@@ -9,5 +9,5 @@
   <child link="chest_1"/>
   <axis xyz="0.0 0.0 1.0"/>
-  <limit upper="0.47" lower="0.00" effort="1000000" velocity="0.5"/>
+  <limit upper="0.201" lower="0.2" effort="1000000" velocity="0.5"/>
 </joint>
 <link name="stand">
